Commit message: typos

File: sedna_description/urdf/sedna.urdf.xacro (robot description, xacro)
@@ -12,5 +12,5 @@
   <xacro:property name="imu_stdev" value="0.00017" />
   <xacro:property name="body_height" value="0.15"/>
-  <xacro:property name="body_length" value="0.38"/>
+  <xacro:property name="body_length" value="0.572"/>
   <xacro:property name="body_width" value="0.32"/>
   <xacro:property name="axis_front" value="0.14"/>

Commit message: adapt wheel radius for smaller wheel

File: sedna_description/urdf/sedna.urdf.xacro (robot description, xacro)
@@ -18,5 +18,5 @@
   <xacro:property name="wheel_thickness" value="0.085"/>
   <xacro:property name="wheel_body_offset" value="${wheel_thickness/2 + 0.015}"/>
-  <xacro:property name="wheel_radius" value="0.135"/>
+  <xacro:property name="wheel_radius" value="0.11"/>
   <xacro:property name="axis_height" value="-0.03"/>
   <xacro:property name="axis_left" value="${-body_width/2 - wheel_body_offset}"/>

Commit message: Made Sedna beautiful and fixed things

File: sedna_description/urdf/sedna.urdf.xacro (robot description, xacro)
@@ -14,7 +14,8 @@
   <xacro:property name="body_length" value="0.572"/>
   <xacro:property name="body_width" value="0.32"/>
-  <xacro:property name="axis_front" value="0.14"/>
-  <xacro:property name="axis_back" value="-0.14"/>
-  <xacro:property name="wheel_thickness" value="0.085"/>
+  <xacro:property name="axis_front" value="0.24"/>
+  <xacro:property name="axis_middle" value="0.0"/>
+  <xacro:property name="axis_back" value="-0.24"/>
+  <xacro:property name="wheel_thickness" value="0.06"/>
   <xacro:property name="wheel_body_offset" value="${wheel_thickness/2 + 0.015}"/>
   <xacro:property name="wheel_radius" value="0.11"/>
@@ -79,8 +80,15 @@
           <!--mesh filename="package://pluto_description/meshes/pluto_wheel.stl"/-->
 	  <cylinder length="${wheel_thickness}" radius="${wheel_radius}"/>
+	  <cylinder length="${wheel_thickness + 0.01} radius=$wheel_radius -0.02}"/>
         </geometry>
         <material name="black" >
           <color rgba="0 0 0 1" />
         </material>
+	<geometry>
+	  <cylinder length="${wheel_thickness + 0.01} radius=$wheel_radius -0.02}"/>
+	</geometry>
+	<material name="red">
+	  <color rgba="1 0 0 1"/>
+	</material>
       </visual>
       <collision>
@@ -96,4 +104,26 @@
         mass="${wheel_mass}" />
     </link>
+    <link name="${name}_link_inner">
+      <visual>
+	<origin xyz="0 0 0" rpy="${M_PI/2} 0 0" />
+        <geometry>
+          <!--mesh filename="package://pluto_description/meshes/pluto_wheel.stl"/-->
+          <cylinder length="${wheel_thickness + 0.01}" radius="${wheel_radius -0.06}"/>
+        </geometry>
+        <material name="red">
+          <color rgba="1 0 0 1"/>
+        </material>
+      </visual>
+	<xacro:cylinder_inertial
+        radius="${wheel_radius -0.02}"
+        length="${wheel_thickness + 0.01}"
+        mass="${wheel_mass}" />
+    </link>
+    <joint name="${name}_joint_inner" type="fixed">
+      <origin xyz="0 0 0" rpy="0 0 0"/>
+      <parent link="${name}_link"/>
+      <child link="${name}_link_inner"/>
+      <axis xyz="0 1 0"/>
+    </joint>
     <joint name="${name}_joint" type="fixed">
       <origin xyz="${xyz}" rpy="0 0 0"/>
@@ -132,4 +162,12 @@
     parent="base_link"
     xyz="${axis_back} ${axis_left} ${axis_height}" />
+  <xacro:wheel
+    name="left_middle_wheel"
+    parent="base_link"
+    xyz="${axis_middle} ${axis_left} ${axis_height}" />
+  <xacro:wheel
+    name="right_middle_wheel"
+    parent="base_link"
+    xyz="${axis_middle} ${axis_right} ${axis_height}" /> i
   <xacro:wheel
     name="right_front_wheel"
